Commit message: Launch gazebo is finished

File: navibot_ws/src/navibot_description/urdf/navibot.urdf.xacro (robot description, xacro)
@@ -2,4 +2,11 @@
 <robot name="navibot" xmlns:xacro="http://ros.org/wiki/xacro">
   <xacro:include filename="$(find navibot_description)/urdf/navibot_gazebo.xacro" />
+  <!-- Material definitions -->
+  <material name="grey">
+    <color rgba="0.2 0.2 0.2 1.0"/>
+  </material>
+  <material name="dark_grey">
+    <color rgba="0.15 0.15 0.15 1.0"/>
+  </material>
   <link name="base_footprint"/>
   <link name="base_link">
@@ -16,4 +23,5 @@
         <mesh filename="package://navibot_description/meshes/base_link.STL" />
       </geometry>
+      <material name="grey"/>
     </visual>
     <collision>
@@ -42,4 +50,5 @@
         <mesh filename="package://navibot_description/meshes/wheel_right_link.STL" />
       </geometry>
+      <material name="dark_grey"/>
     </visual>
     <collision>
@@ -70,4 +79,5 @@
         <mesh filename="package://navibot_description/meshes/wheel_left_link.STL" />
       </geometry>
+      <material name="dark_grey"/>
     </visual>
     <collision>
@@ -97,4 +107,5 @@
         <mesh filename="package://navibot_description/meshes/caster_front_link.STL" />
       </geometry>
+      <material name="grey"/>
     </visual>
     <collision>
@@ -124,4 +135,5 @@
         <mesh filename="package://navibot_description/meshes/caster_rear_link.STL" />
       </geometry>
+      <material name="grey"/>
     </visual>
     <collision>
